Commit message: Added two node:
-odom: uses topic /high_state to generate odometry data
-imu: uses topic /high_state to generate sensor mesage::imu

both topics are published via udp

File: go1_robot_description/xacro/depthCamera.xacro (robot description, xacro)
@@ -4,5 +4,5 @@
         <joint name="camera_joint_${name}" type="fixed">
             <xacro:insert_block name="origin"/>
-            <parent link="trunk"/>
+            <parent link="base_link"/>
             <child link="camera_${name}"/>
         </joint>

File: go1_robot_description/xacro/leg.xacro (robot description, xacro)
@@ -16,5 +16,5 @@
                 <origin rpy="0 0 0" xyz="${-leg_offset_x} ${leg_offset_y} 0"/>
             </xacro:if>
-            <parent link="trunk"/>
+            <parent link="base_link"/>
             <child link="${name}_hip"/>
             <axis xyz="1 0 0"/>
@@ -40,5 +40,5 @@
                 <origin rpy="0 0 0" xyz="${-hip_rotor_offset_x} ${hip_rotor_offset_y} 0"/>
             </xacro:if>
-            <parent link="trunk"/>
+            <parent link="base_link"/>
             <child link="${name}_hip_rotor"/>
         </joint>

File: go1_robot_description/xacro/robot.xacro (robot description, xacro)
@@ -22,5 +22,11 @@
         </joint>
     </xacro:if>
-    <link name="base_link">
+    <!-- <link name="odom"/>
+    <joint name="odom_base" type="fixed">
+        <origin rpy="0 0 0" xyz="0 0 0"/>
+        <parent link="odom"/>
+        <child link="base_link"/>
+    </joint> -->
+    <link name="world">
         <visual>
             <origin rpy="0 0 0" xyz="0 0 0"/>
@@ -30,12 +36,12 @@
         </visual>
     </link>
-    <joint name="floating_base" type="fixed">
+    <joint name="world_to_mybase_link" type="fixed">
         <origin rpy="0 0 0" xyz="0 0 0"/>
-        <parent link="base_link"/>
-        <child link="trunk"/>
+        <parent link="world"/>
+        <child link="base_link"/>
     </joint>
-    <link name="trunk">
+    <link name="base_link">
         <visual>
-            <origin rpy="0 0 0" xyz="0 0 0"/>
+            <origin rpy="0 0 0" xyz="0 0 0.1"/>
             <geometry>
                 <mesh filename="package://go1_robot_description/meshes/trunk.dae" scale="1 1 1"/>
@@ -67,10 +73,10 @@
     </link>
     <joint name="lidar_joint" type="fixed">
-        <origin rpy="0 0 0.1" xyz="0 0 0"/>
-        <parent link="trunk"/>
+        <origin rpy="0 0 0" xyz="0.3 0 0.15"/>
+        <parent link="base_link"/>
         <child link="rslidar"/>
     </joint>
     <joint name="imu_joint" type="fixed">
-        <parent link="trunk"/>
+        <parent link="base_link"/>
         <child link="imu_link"/>
         <origin rpy="0 0 0" xyz="-0.01592 -0.06659 -0.00617"/>

File: go1_robot_description/xacro/robot_simple.xacro (robot description, xacro)
@@ -2,5 +2,4 @@
 <robot name="go1" xmlns:xacro="http://www.ros.org/wiki/xacro">
     <xacro:arg name="DEBUG" default="false"/>
-    <!-- Actually, the rotor will rotate and the joint is not fixed. Reduction ratio should be considered. -->
     <!-- Debug mode will hung up the robot, use "true" or "false" to switch it. -->
     <xacro:if value="$(arg DEBUG)">
@@ -12,40 +11,11 @@
         </joint>
     </xacro:if>
-<!--
-    <link name="base">
+    <link name="base_link">
         <visual>
             <origin rpy="0 0 0" xyz="0 0 0"/>
             <geometry>
-                <box size="0.001 0.001 0.001"/>
+                <box size="0.1 0.1 0.1"/>
             </geometry>
         </visual>
-    </link>
-    <joint name="floating_base" type="fixed">
-        <origin rpy="0 0 0" xyz="0 0 0"/>
-        <parent link="base_link"/>
-        <child link="trunk"/>
-    </joint> -->
-    <link name="trunk">
-        <visual>
-            <origin rpy="0 0 0" xyz="0 0 0"/>
-            <geometry>
-                <mesh filename="package://go1_robot_description/meshes/trunk.dae" scale="1 1 1"/>
-            </geometry>
-            <!-- <material name="orange"/> -->
-        </visual>
-        <collision>
-            <origin rpy="0 0 0" xyz="0 0 0"/>
-            <geometry>
-                <box size="${trunk_length} ${trunk_width} ${trunk_height}"/>
-            </geometry>
-        </collision>
-        <inertial>
-            <origin rpy="0 0 0" xyz="${trunk_com_x} ${trunk_com_y} ${trunk_com_z}"/>
-            <mass value="${trunk_mass}"/>
-            <inertia
-                ixx="${trunk_ixx}" ixy="${trunk_ixy}" ixz="${trunk_ixz}"
-                iyy="${trunk_iyy}" iyz="${trunk_iyz}"
-                izz="${trunk_izz}"/>
-        </inertial>
     </link>
     <link name="rslidar">
@@ -58,7 +28,32 @@
     </link>
     <joint name="lidar_joint" type="fixed">
-        <origin rpy="0 0 0.1" xyz="0 0 0"/>
-        <parent link="trunk"/>
+        <origin rpy="0 0 0" xyz="0.3 0 0.15"/>
+        <parent link="base_link"/>
         <child link="rslidar"/>
     </joint>
+<joint name="imu_joint" type="fixed">
+        <parent link="base_link"/>
+        <child link="imu_link"/>
+        <origin rpy="0 0 0" xyz="-0.01592 -0.06659 -0.00617"/>
+    </joint>
+    <link name="imu_link">
+        <inertial>
+            <mass value="0.001"/>
+            <origin rpy="0 0 0" xyz="0 0 0"/>
+            <inertia ixx="0.0001" ixy="0" ixz="0" iyy="0.0001" iyz="0" izz="0.0001"/>
+        </inertial>
+        <visual>
+            <origin rpy="0 0 0" xyz="0 0 0"/>
+            <geometry>
+                <box size="0.001 0.001 0.001"/>
+            </geometry>
+            <!-- <material name="red"/> -->
+        </visual>
+        <collision>
+            <origin rpy="0 0 0" xyz="0 0 0"/>
+            <geometry>
+                <box size=".001 .001 .001"/>
+            </geometry>
+        </collision>
+    </link>
 </robot>

File: go1_robot_description/xacro/ultraSound.xacro (robot description, xacro)
@@ -4,5 +4,5 @@
         <joint name="ultraSound_joint_${name}" type="fixed">
             <xacro:insert_block name="origin"/>
-            <parent link="trunk"/>
+            <parent link="base_link"/>
             <child link="ultraSound_${name}"/>
         </joint>
